File: flash.kicad_sch (KiCad schematic)
At the start: 15 parts, among them IC1 IS42S16160J-6BLI, IC2 S26KL512SDABHV020, U1 MIMXRT1052CVJ5B

Commit message: v0.2
Parts:
- C38: value 100nF -> DNP
Connections:
- net LPI2C3_SDA: now reaches U1.J3 (GPIO_SD_B0_01)
- net LPI2C3_SCL: now reaches U1.J4 (GPIO_SD_B0_00)
- net ENET_MDC: no longer names the net of U1.A7 (GPIO_EMC_40)
- net ENET_MDIO: no longer names the net of U1.C7 (GPIO_EMC_41)
Other:
- title: RT1050 DevBoard for Project Horizon -> Payload Board for Pleiades Atlas
- moved on the sheet: C39, C40, IC2, R2, R3
