File: usb_debug.kicad_sch (KiCad schematic)
At the start: 19 parts, among them J5 USB_C_Receptacle_USB2.0, SW1 SW_DIP_x02, U1 MIMXRT1052CVJ5B, U7 PRTR5V0U2X, U8 XC6206P332PR-G

Commit message: v0.2
Parts:
- removed C53, C54: 1uF, Capacitor_SMD:C_0201_0603Metric, symbol Device:C_Small
- removed R13, R14, R15: 1k, Resistor_SMD:R_0402_1005Metric, symbol Device:R_Small_US
- removed R16, R17, R18: 10k, Resistor_SMD:R_0402_1005Metric, symbol Device:R_Small_US
- removed SW1: SW_DIP_x02, Button_Switch_SMD:SW_DIP_SPSTx02_Slide_6.7x6.64mm_W6.73mm_P2.54mm_LowProfile_JPin, symbol Switch:SW_DIP_x02
- removed U8: XC6206P332PR-G, Package_TO_SOT_SMD:SOT-23, symbol kicad-keyboard-parts:XC6206PxxxMR-Regulator_Linear
- added C45, C49: 0.1uF, symbol Device:C_Small
- added C46, C55, C63, C64, C65, C66, C68: C_100n_16V_X7R_0402, antmicro-footprints:C_0402_1005Metric, symbol antmicroCapacitors0402:C_100n_16V_X7R_0402
- added C47, C48: 10pF, symbol Device:C_Small
- added C56, C57, C67: C_4u7_0402, antmicro-footprints:C_0402_1005Metric, symbol antmicroCapacitors0402:C_4u7_0402
- added FB1, FB2: FB_600Z_0.3A_Murata-BLM15AG_0402, antmicro-footprints:FB_0402_1005Metric, symbol antmicroFerriteBeadsandChips:FB_600Z_0.3A_Murata-BLM15AG_0402
- added IC3: 93LC66BT-I_MC, SON50P300X200X100-9N-D, symbol 93LC66BT-I_MC:93LC66BT-I_MC
- added J1: USB_C_Receptacle_USB2.0, Connector_USB:USB_C_Receptacle_HRO_TYPE-C-31-M-12, symbol Connector:USB_C_Receptacle_USB2.0
- added L3: 60R@100MHz, Inductor_SMD:L_1206_3216Metric, symbol Unified-Daughterboard-rescue:L_Core_Ferrite-Device
- added R10, R20, R6, R9: 10k, symbol Device:R_US
- added R11: 2.2k, symbol Device:R_US
- added R12, R19: 5.1k, Resistor_SMD:R_0402_1005Metric, symbol Device:R_US
- added R21: 12k, symbol Device:R_US
- added U5: FT2232HQ, Package_DFN_QFN:QFN-64-1EP_9x9mm_P0.5mm_EP4.35x4.35mm, symbol Interface_USB:FT2232HQ
- added Y3: 830105420809, 830105420809, symbol 830105420809:830105420809
Connections:
- net +3.3V: now also C45.1, IC3.8 (VCC), R10.1, R20.1, R6.1, R9.1
- net GND: now also C45.2, C46.2, C47.2, C48.2, C49.2, C55.2, C56.2, C57.1, C63.2, C64.2, C65.2, C66.1, C67.2, C68.2, IC3.5 (VSS_1), IC3.9 (VSS_2), R12.1, R19.1, R21.1, U5.1 (GND), U5.10 (AGND), U5.11 (GND), U5.13 (TEST), U5.15 (GND), U5.25 (GND), U5.35 (GND), U5.47 (GND), U5.5 (GND), U5.51 (GND), U5.65 (GND), Y3.2 (GND_&_LID_1), Y3.4 (GND_&_LID_2)
- new net: C49.1, R20.2, U5.14 (~{RESET})
- new net: J1.A1 (GND), J1.A12 (GND), J1.B1 (GND), J1.B12 (GND), J1.S1 (SHIELD), L3.1, L3.2
- new net: J1.A5 (CC1), R12.2
- new net: J1.B5 (CC2), R19.2
- new net: R21.2, U5.6 (REF)
- new net: IC3.4 (DO), R11.2
- new net +1V8A: C63.1, C67.1, U5.12 (VCORE), U5.37 (VCORE), U5.49 (VREGOUT), U5.64 (VCORE)
- new net +3V3: C46.1, C55.1, C64.1, C68.1, FB1.1, FB2.1, U5.20 (VCCIO), U5.31 (VCCIO), U5.42 (VCCIO), U5.50 (VREGIN), U5.56 (VCCIO)
- new net DM_DEBUG: J1.A7 (D-), J1.B7 (D-), U5.7 (DM)
- new net DP_DEBUG: J1.A6 (D+), J1.B6 (D+), U5.8 (DP)
- new net EECLK: IC3.2 (CLK), R9.2, U5.62 (EECLK)
- new net EECS: IC3.1 (CS), R10.2, U5.63 (EECS)
- new net EEDATA: IC3.3 (DI), R11.1, R6.2, U5.61 (EEDATA)
- new net JTAG_TCK: U5.16 (ADBUS0)
- new net JTAG_TDI: U5.17 (ADBUS1)
- new net JTAG_TDO: U5.18 (ADBUS2)
- new net JTAG_TMS: U5.19 (ADBUS3)
- new net JTAG_TRSTB: U5.28 (ACBUS2)
- new net LPUART2_RX: U5.39 (BDBUS1)
- new net LPUART2_TX: U5.38 (BDBUS0)
- new net VBUS_FTDI: J1.A4 (VBUS), J1.A9 (VBUS), J1.B4 (VBUS), J1.B9 (VBUS)
- new net VPHY: C56.1, C65.1, FB1.2, U5.4 (VPHY)
- new net VPLL: C57.2, C66.2, FB2.2, U5.9 (VPLL)
- new net XCSI: C47.1, U5.2 (OSCI), Y3.1 (CRYSTAL_1)
- new net XCSO: C48.1, U5.3 (OSCO), Y3.3 (CRYSTAL_2)
- no-connect marks 6 -> 37
Other:
- title: RT1050 DevBoard for Project Horizon -> Payload Board for Pleiades Atlas

Commit message: started layout
Parts:
- added CR1, CR2: CMS04TE12L_Q_M, M-FLAT_TOS, symbol CMS04(TE12L,Q,M):CMS04TE12L_Q_M
- C45, C47, C48, C49: footprint (none) -> Capacitor_SMD:C_0201_0603Metric
- C46, C55, C56, C57, C63, C64, C65, C66, C67, C68: footprint antmicro-footprints:C_0402_1005Metric -> Capacitor_SMD:C_0402_1005Metric
- FB1, FB2: footprint antmicro-footprints:FB_0402_1005Metric -> Inductor_SMD:L_0402_1005Metric
- R10, R11, R20, R21, R6, R9: footprint (none) -> Resistor_SMD:R_0402_1005Metric
Connections:
- net +5V: now also CR1.2; no longer J5.A4 (VBUS), J5.A9 (VBUS), J5.B4 (VBUS), J5.B9 (VBUS)
- net VBUS_FTDI: now also CR2.2; no longer J1.A4 (VBUS), J1.A9 (VBUS), J1.B4 (VBUS), J1.B9 (VBUS)
- new net: CR2.1, J1.A4 (VBUS), J1.A9 (VBUS), J1.B4 (VBUS), J1.B9 (VBUS)
- new net: CR1.1, J5.A4 (VBUS), J5.A9 (VBUS), J5.B4 (VBUS), J5.B9 (VBUS)
Other:
- moved on the sheet: J5, L2, R7, R8

Commit message: finished layout of v0.2!
Parts:
- added U14: PRTR5V0U2X, Package_TO_SOT_SMD:SOT-143, symbol Power_Protection:PRTR5V0U2X
Connections:
- net VBUS_FTDI is gone; now on net +5V: CR2.2
- net +5V: now also U14.4 (VCC)
- net DM_DEBUG: now also U14.2 (I/O1)
- net DP_DEBUG: now also U14.3 (I/O2)
- net GND: now also J1.A1 (GND), J1.A12 (GND), J1.B1 (GND), J1.B12 (GND), J1.S1 (SHIELD), L3.1, L3.2, U14.1 (GND)
