File: RT1050.kicad_pcb (KiCad board)
At the start: 4 copper layers, 88 x 94.5 mm, 113 parts, among them IC1 IS42S16160J-6BLI, IC2 S26KL512SDABHV020, J1 Conn_01x04_Pin, J10 Conn_01x06_Pin, J13 Conn_02x04_Counter_Clockwise, J14 Conn_02x04_Counter_Clockwise, J2 Conn_01x04_Pin, J3 Conn_01x20, J4 Conn_01x05_Pin, J5 USB_C_Receptacle_USB2.0, J6 Conn_01x02, J7 Conn_01x02, J8 Conn_Coaxial_Small, J9 Conn_01x04_Pin, SW1 SW_DIP_x02, U1 MIMXRT1052CVJ5B, U10 TPS22921YZPR, U11 TPS22921YZPR, U12 CY15B064J-SXET, U2 DP83TC813SRHFRQ1, U3 MMC5983MA, U4 BMI088, U5 RFM98W-433S2, U6 TCAN334, U7 PRTR5V0U2X, U8 XC6206P332PR-G, U9 MCP23009-E/MG, Y1 DSC1001BI5-024.0000, Y2 830107834801

Commit message: v0.2
Connections:
- U2 pad 28: unconnected-(U2-RX_CLK-Pad28) -> (no net)
Routing:
- net SPE_V: vias 7 -> 6
- net (no net): vias 0 -> 1
- added copper zone on In1.Cu, net (none)
- removed copper zone on In1.Cu, net SPE_V

Commit message: started layout
Parts:
- removed FL1: DLW32MH201XK2L, footprints:DLW32MH101XK2L
- removed G***: LOGO, LOGO
- removed J13, J14: Conn_02x04_Counter_Clockwise, Connector_PinHeader_2.00mm:PinHeader_2x04_P2.00mm_Vertical
- removed SW1: SW_DIP_x02, Button_Switch_SMD:SW_DIP_SPSTx02_Slide_6.7x6.64mm_W6.73mm_P2.54mm_LowProfile_JPin
- removed U11: TPS22921YZPR, footprints:YZP6
- removed U2: DP83TC813SRHFRQ1, footprints:VQFN28_RHF_TEX
- removed U8: XC6206P332PR-G, Package_TO_SOT_SMD:SOT-23
- removed U9: MCP23009-E/MG, footprints:QFN16_3x3MC_MCH
- added C63: C_100n_16V_X7R_0402, Capacitor_SMD:C_0402_1005Metric, F.Cu at (199.4, 77.3)
- added C64: C_100n_16V_X7R_0402, Capacitor_SMD:C_0402_1005Metric, F.Cu at (202.3, 69.4)
- added C65: C_100n_16V_X7R_0402, Capacitor_SMD:C_0402_1005Metric, F.Cu at (202.3, 71.4)
- added C66: C_100n_16V_X7R_0402, Capacitor_SMD:C_0402_1005Metric, F.Cu at (202.3, 73.4)
- added C67: C_4u7_0402, Capacitor_SMD:C_0402_1005Metric, F.Cu at (202.3, 75.3)
- added C68: C_100n_16V_X7R_0402, Capacitor_SMD:C_0402_1005Metric, F.Cu at (202.3, 77.3)
- added C69: 22nF, Capacitor_SMD:C_0201_0603Metric, F.Cu at (265.0, 53.2)
- added C70: 4.7uF, Capacitor_SMD:C_0201_0603Metric, F.Cu at (265.0, 55.0)
- added C71: 0.22uF, Capacitor_SMD:C_0201_0603Metric, F.Cu at (265.0, 56.7)
- added C72: 10u, Capacitor_SMD:C_0603_1608Metric, F.Cu at (233.7, 96.1)
- added C73: 100nf, Capacitor_SMD:C_0402_1005Metric, F.Cu at (224.4, 109.8)
- added C74: 10u, Capacitor_SMD:C_0603_1608Metric, F.Cu at (233.7, 98.6)
- added C75: 100nf, Capacitor_SMD:C_0402_1005Metric, F.Cu at (224.4, 111.7)
- added C76: 10u, Capacitor_SMD:C_0603_1608Metric, F.Cu at (233.7, 101.1)
- added C77: 10u, Capacitor_SMD:C_0603_1608Metric, F.Cu at (233.7, 103.6)
- added C78: 10u, Capacitor_SMD:C_0603_1608Metric, F.Cu at (233.7, 106.1)
- added C79: 22nF, Capacitor_SMD:C_0201_0603Metric, F.Cu at (267.5, 53.2)
- added C80: 0.22uF, Capacitor_SMD:C_0201_0603Metric, F.Cu at (267.5, 55.0)
- added C81: 4.7uF, Capacitor_SMD:C_0201_0603Metric, F.Cu at (267.5, 56.7)
- added C82: 22nF, Capacitor_SMD:C_0201_0603Metric, F.Cu at (269.9, 53.2)
- added C83: 0.22uF, Capacitor_SMD:C_0201_0603Metric, F.Cu at (269.9, 55.0)
- added C84: 4.7uF, Capacitor_SMD:C_0201_0603Metric, F.Cu at (269.9, 56.7)
- added C85: 100nf, Capacitor_SMD:C_0402_1005Metric, F.Cu at (265.2, 58.6)
- added C86: 100nf, Capacitor_SMD:C_0402_1005Metric, F.Cu at (265.2, 60.6)
- added CR1: CMS04TE12L_Q_M, footprints:M-FLAT_TOS, F.Cu at (244.0, 65.7)
- added CR2: CMS04TE12L_Q_M, footprints:M-FLAT_TOS, F.Cu at (244.0, 69.7)
- added D6: GREEN, LED_SMD:LED_0603_1608Metric, F.Cu at (237.8, 102.6)
- added D7: 1N4151WS, Diode_SMD:D_SOD-323, F.Cu at (237.9, 99.9)
- added FB1: FB_600Z_0.3A_Murata-BLM15AG_0402, Inductor_SMD:L_0402_1005Metric, F.Cu at (205.2, 69.5)
- added FB2: FB_600Z_0.3A_Murata-BLM15AG_0402, Inductor_SMD:L_0402_1005Metric, F.Cu at (205.2, 71.4)
- added H1: MountingHole, , F.Cu at (32.4, 141.5)
- added H2: MountingHole, , F.Cu at (112.4, 141.5)
- added IC3: 93LC66BT-I_MC, footprints:SON50P300X200X100-9N-D, F.Cu at (237.3, 75.7)
- added J11: Conn_01x02_Pin, Connector_JST:JST_SH_BM02B-SRSS-TB_1x02-1MP_P1.00mm_Vertical, F.Cu at (254.6, 68.0)
- added JP6: SolderJumper_2_Open, Jumper:SolderJumper-2_P1.3mm_Open_RoundedPad1.0x1.5mm, F.Cu at (237.9, 96.6)
- added L3: 60R@100MHz, Inductor_SMD:L_1206_3216Metric, F.Cu at (243.4, 77.0)
- added L4: 2.2uH, Resistor_SMD:R_0402_1005Metric, F.Cu at (276.7, 82.2)
- added R19: 5.1k, Resistor_SMD:R_0402_1005Metric, F.Cu at (239.1, 68.6)
- added R20: 10k, Resistor_SMD:R_0402_1005Metric, F.Cu at (239.1, 70.6)
- added R21: 12k, Resistor_SMD:R_0402_1005Metric, F.Cu at (239.1, 72.6)
- added R22: 10k, Resistor_SMD:R_0402_1005Metric, F.Cu at (277.1, 64.5)
- added R23: 120k, Resistor_SMD:R_0402_1005Metric, F.Cu at (259.4, 57.3)
- added R24: 2.2k, Resistor_SMD:R_0402_1005Metric, F.Cu at (259.4, 59.3)
- added R25: 10k, Resistor_SMD:R_0402_1005Metric, F.Cu at (224.4, 89.8)
- added R26: 10k, Resistor_SMD:R_0402_1005Metric, F.Cu at (224.4, 91.8)
- added R27: 10k, Resistor_SMD:R_0402_1005Metric, F.Cu at (243.9, 82.2)
- added R28: 10k, Resistor_SMD:R_0402_1005Metric, F.Cu at (243.9, 84.1)
- added R29: 10k, Resistor_SMD:R_0402_1005Metric, F.Cu at (243.9, 86.1)
- added R30: 10k, Resistor_SMD:R_0402_1005Metric, F.Cu at (243.9, 88.1)
- added R31: 10k, Resistor_SMD:R_0402_1005Metric, F.Cu at (243.9, 90.1)
- added R32: 10k, Resistor_SMD:R_0402_1005Metric, F.Cu at (243.9, 92.1)
- added R33: 10k, Resistor_SMD:R_0402_1005Metric, F.Cu at (243.9, 94.1)
- added R34: 10k, Resistor_SMD:R_0402_1005Metric, F.Cu at (246.8, 82.2)
- added R35: 10k, Resistor_SMD:R_0402_1005Metric, F.Cu at (246.8, 84.1)
- added R36: 10k, Resistor_SMD:R_0402_1005Metric, F.Cu at (246.8, 86.1)
- added R37: 10k, Resistor_SMD:R_0402_1005Metric, F.Cu at (246.8, 88.1)
- added R38: 10k, Resistor_SMD:R_0402_1005Metric, F.Cu at (246.8, 90.1)
- added R39: 10k, Resistor_SMD:R_0402_1005Metric, F.Cu at (246.8, 92.1)
- added R40: 10k, Resistor_SMD:R_0402_1005Metric, F.Cu at (246.8, 94.1)
- added R41: 1k, Resistor_SMD:R_0402_1005Metric, F.Cu at (249.8, 82.2)
- added R42: 1k, Resistor_SMD:R_0402_1005Metric, F.Cu at (249.8, 84.1)
- added R43: 1k, Resistor_SMD:R_0402_1005Metric, F.Cu at (249.8, 86.1)
- added R44: 1k, Resistor_SMD:R_0402_1005Metric, F.Cu at (249.8, 88.1)
- added R45: 3.0k, Resistor_SMD:R_0402_1005Metric, F.Cu at (224.4, 101.8)
- added R46: 3.0k, Resistor_SMD:R_0402_1005Metric, F.Cu at (224.4, 103.8)
- added R47: 3.0k, Resistor_SMD:R_0402_1005Metric, F.Cu at (224.4, 105.8)
- added R48: 10k, Resistor_SMD:R_0402_1005Metric, F.Cu at (224.4, 107.8)
- added R49: 10k, Resistor_SMD:R_0402_1005Metric, F.Cu at (227.4, 95.8)
- added R50: 47k, Resistor_SMD:R_0402_1005Metric, F.Cu at (227.4, 97.8)
- added R51: 1k, Resistor_SMD:R_0402_1005Metric, F.Cu at (227.4, 99.8)
- added R52: 100k, Resistor_SMD:R_0402_1005Metric, F.Cu at (227.4, 101.8)
- added R53: 1k, Resistor_SMD:R_0402_1005Metric, F.Cu at (227.4, 103.8)
- added R54: 100k, Resistor_SMD:R_0402_1005Metric, F.Cu at (227.4, 105.8)
- added R55: 100k, Resistor_SMD:R_0402_1005Metric, F.Cu at (227.4, 107.8)
- added R56: 100k, Resistor_SMD:R_0402_1005Metric, F.Cu at (230.3, 95.8)
- added R57: 4.7M, Resistor_SMD:R_0402_1005Metric, F.Cu at (230.3, 97.8)
- added R58: 100k, Resistor_SMD:R_0402_1005Metric, F.Cu at (230.3, 99.8)
- added R59: 100k, Resistor_SMD:R_0402_1005Metric, F.Cu at (230.3, 101.8)
- added R60: 120k, Resistor_SMD:R_0402_1005Metric, F.Cu at (259.4, 61.3)
- added R61: 2.2k, Resistor_SMD:R_0402_1005Metric, F.Cu at (262.3, 53.4)
- added R62: 120k, Resistor_SMD:R_0402_1005Metric, F.Cu at (262.3, 55.4)
- added R63: 2.2k, Resistor_SMD:R_0402_1005Metric, F.Cu at (262.3, 57.3)
- added R64: 330m, Resistor_SMD:R_0402_1005Metric, F.Cu at (262.3, 59.3)
- added R65: 47k, Resistor_SMD:R_0402_1005Metric, F.Cu at (262.3, 61.3)
- added SW2: SW_DIP_x04, Button_Switch_SMD:SW_DIP_SPSTx04_Slide_Copal_CHS-04A_W5.08mm_P1.27mm_JPin, F.Cu at (255.3, 85.2)
- added VR1: TS53YJ203MR10, footprints:TS53YJ203MR10, F.Cu at (262.0, 66.9)
- added Y3: 830105420809, footprints:830105420809, F.Cu at (226.3, 76.2)
- C13, C25, C40, R1: moved to B.Cu
- C27, C29, C33, C34, C49: moved to F.Cu
- C38: value 100nF -> DNP
- C45: value 0.47uF -> 0.1uF
- C46: value 0.01uF -> C_100n_16V_X7R_0402; footprint Capacitor_SMD:C_0201_0603Metric -> Capacitor_SMD:C_0402_1005Metric
- C47: value 0.47uF -> 10pF
- C48: value 0.01uF -> 10pF
- C53: value 1uF -> 10uF; footprint Capacitor_SMD:C_0201_0603Metric -> Capacitor_SMD:C_0402_1005Metric
- C54: value 1uF -> 22uF; footprint Capacitor_SMD:C_0201_0603Metric -> Capacitor_SMD:C_0603_1608Metric
- C55: value 100nF -> C_100n_16V_X7R_0402; footprint Capacitor_SMD:C_0201_0603Metric -> Capacitor_SMD:C_0402_1005Metric
- C56: value 100nF -> C_4u7_0402; footprint Capacitor_SMD:C_0201_0603Metric -> Capacitor_SMD:C_0402_1005Metric
- C57: value 4.7n -> C_4u7_0402; footprint Capacitor_SMD:C_0201_0603Metric -> Capacitor_SMD:C_0402_1005Metric; moved to F.Cu
- J1: value Conn_01x04_Pin -> USB_C_Receptacle_USB2.0; footprint Connector_PinHeader_2.00mm:PinHeader_1x04_P2.00mm_Vertical -> Connector_USB:USB_C_Receptacle_HRO_TYPE-C-31-M-12
- J10: value Conn_01x06_Pin -> Conn_01x02_Pin; footprint Connector_PinHeader_2.00mm:PinHeader_1x06_P2.00mm_Vertical -> Connector_JST:JST_SH_BM02B-SRSS-TB_1x02-1MP_P1.00mm_Vertical
- J2: value Conn_01x04_Pin -> Conn_01x03_Pin; footprint Connector_PinHeader_2.00mm:PinHeader_1x04_P2.00mm_Vertical -> Connector_PinHeader_1.00mm:PinHeader_1x03_P1.00mm_Vertical
- J3: footprint Connector_FFC-FPC:Molex_200528-0200_1x20-1MP_P1.00mm_Horizontal -> Connector_FFC-FPC:TE_2-1734839-0_1x20-1MP_P0.5mm_Horizontal
- J4: value Conn_01x05_Pin -> Conn_01x03_Pin; footprint Connector_PinHeader_2.00mm:PinHeader_1x04_P2.00mm_Vertical -> Connector_PinHeader_1.00mm:PinHeader_1x03_P1.00mm_Vertical
- J6: value Conn_01x02 -> Conn_01x02_Pin; footprint Connector_JST:JST_SH_BM02B-SRSS-TB_1x02-1MP_P1.00mm_Vertical -> Connector_PinHeader_1.00mm:PinHeader_1x02_P1.00mm_Vertical
- J7: value Conn_01x02 -> Conn_01x02_Pin; footprint Connector_JST:JST_PH_B2B-PH-K_1x02_P2.00mm_Vertical -> Connector_PinHeader_1.00mm:PinHeader_1x02_P1.00mm_Vertical
- J8: value Conn_Coaxial_Small -> Conn_01x04_Pin; footprint Connector_Coaxial:SMA_Amphenol_132134_Vertical -> Connector_PinHeader_1.00mm:PinHeader_1x04_P1.00mm_Vertical
- J9: value Conn_01x04_Pin -> Conn_01x02_Pin; footprint Connector_PinHeader_2.00mm:PinHeader_1x04_P2.00mm_Vertical -> Connector_JST:JST_SH_BM02B-SRSS-TB_1x02-1MP_P1.00mm_Vertical
- R10, R9: value 1k -> 10k; moved to F.Cu
- R11: value 100k -> 2.2k; moved to F.Cu
- R12: value 10k -> 5.1k; moved to F.Cu
- R13: value 1k -> 100k
- R14, R15: value 1k -> 330m
- R6: value 120 -> 10k
- U10: value TPS22921YZPR -> TPS62162DSG; footprint footprints:YZP6 -> Package_SON:WSON-8-1EP_2x2mm_P0.5mm_EP0.9x1.6mm_ThermalVias
- U5: value RFM98W-433S2 -> FT2232HQ; footprint footprints:HOPERF_RFM95W_SMD -> Package_DFN_QFN:QFN-64-1EP_9x9mm_P0.5mm_EP4.35x4.35mm
- U6: value TCAN334 -> TLV1704; footprint footprints:DCN0008A_M -> Package_SO:TSSOP-14_4.4x5mm_P0.65mm
- moved C43 207.1 mm to (274.2, 107.0), turned to 0 degrees
- moved C39 206.5 mm to (271.7, 108.7), turned to 0 degrees
- moved C41 205.3 mm to (274.2, 103.5), turned to 0 degrees
- moved C54 203.3 mm to (273.2, 84.9)
- moved J2 203.0 mm to (278.2, 53.9)
- moved J6 200.7 mm to (278.2, 58.9), turned to 0 degrees
- moved C37 200.2 mm to (271.7, 105.2), turned to 0 degrees
- moved C53 199.6 mm to (275.7, 96.3), turned to 0 degrees
- moved C38 198.7 mm to (271.7, 107.0)
- moved C58 198.5 mm to (274.4, 64.3), turned to 0 degrees
- moved J4 195.4 mm to (281.5, 53.9), turned to 0 degrees
- moved J9 192.3 mm to (254.6, 55.5)
- moved C21 191.1 mm to (267.6, 89.0), turned to 0 degrees
- moved R13 189.9 mm to (276.7, 86.1), turned to 0 degrees
- moved C22 189.9 mm to (267.6, 90.8), turned to 0 degrees
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Connections:
- C45 pad 1: SPE_V -> +3.3V
- C46 pad 1: SPE_V -> +3.3V
- C47 pad 1: SPE_V -> XCSI
- C48 pad 1: SPE_V -> XCSO
- C49 pad 1: SPE_V -> Net-(U5-~{RESET})
- C53 pad 1: GND -> VBUS
- C53 pad 2: VBUS -> GND
- C54 pad 1: GND -> +3.3V
- C54 pad 2: +3.3V -> GND
- C55 pad 1: Net-(C55-Pad1) -> +3.3V
- C55 pad 2: Net-(J7-Pin_1) -> GND
- C56 pad 1: Net-(C56-Pad1) -> /USB & Debug/VPHY
- C56 pad 2: Net-(J7-Pin_2) -> GND
- C57 pad 2: Net-(C57-Pad2) -> /USB & Debug/VPLL
- J10 pad 1: GND -> Net-(J10-Pin_1)
- J10 pad 2: LPSPI4_SCK -> Net-(J10-Pin_2)
- J2 pad 1: GND -> LPSPI3_SCK
- J2 pad 2: LPUART3_RX -> LPSPI3_SDO
- J2 pad 3: LPUART3_TX -> LPSPI3_SDI
- J3 pad 3: LPI2C2_SDA -> LPI2C3_SDA
- J3 pad 4: LPI2C2_SCL -> LPI2C3_SCL
- J4 pad 1: +3.3V -> LPSPI4_SCK
- J4 pad 2: LPI2C1_SDA -> LPSPI4_SDO
- J4 pad 3: LPI2C1_SCL -> LPSPI4_SDI
- J5 pad A4: VBUS -> Net-(CR1-Pad1)
- J5 pad A9: VBUS -> Net-(CR1-Pad1)
- J5 pad B4: VBUS -> Net-(CR1-Pad1)
- J5 pad B9: VBUS -> Net-(CR1-Pad1)
- J6 pad 1: CANH -> LPI2C4_SCL
- J6 pad 2: CANL -> LPI2C4_SDA
- J7 pad 1: Net-(J7-Pin_1) -> GPIO_B0_08
- J7 pad 2: Net-(J7-Pin_2) -> GPIO_B0_09
- J8 pad 1: Net-(J8-In) -> VBUS
- J8 pad 2: GND -> +3.3V
- J9 pad 1: GND -> Net-(J9-Pin_1)
- J9 pad 2: LPUART2_RX -> Net-(J9-Pin_2)
- R10 pad 1: Net-(J7-Pin_2) -> +3.3V
- R10 pad 2: Net-(C57-Pad2) -> EECS
- R11 pad 1: Net-(C57-Pad2) -> EEDATA
- R11 pad 2: GND -> Net-(IC3-DO)
- R12 pad 1: +3.3V -> GND
- R12 pad 2: LPSPI3_CS -> Net-(J1-CC1)
- R13 pad 2: GPIO_B0_13 -> Net-(U10-PG)
- R14 pad 1: +3.3V -> Net-(U2-SENSEA)
- R14 pad 2: Net-(R14-Pad2) -> GND
- R15 pad 1: +3.3V -> Net-(U8-SENSEA)
- R15 pad 2: Net-(R15-Pad2) -> GND
- R16 pad 1: GND -> WDT_BIAS
- R16 pad 2: GPIO_B0_13 -> Net-(R16-Pad2)
- R17 pad 1: GND -> Net-(R16-Pad2)
- R17 pad 2: CSI_DATA_8 -> Net-(U6D--)
- R18 pad 1: GPIO_AD_B0_04 -> Net-(U6D--)
- R18 pad 2: GND -> Net-(U6B--)
- R6 pad 1: CANH -> +3.3V
- R6 pad 2: CANL -> EEDATA
- R9 pad 1: Net-(J7-Pin_1) -> +3.3V
- R9 pad 2: Net-(C57-Pad2) -> EECLK
- U1 pad A10: STB -> GPIO_B0_11
- U1 pad A12: ENET_TX_DATA_1 -> STB
- U1 pad A13: ENET_TX_EN -> SHDN
- U1 pad A7: ENET_MDC -> unconnected-(U1H-GPIO_EMC_40-PadA7)
- U1 pad A8: DIO4 -> GPIO_B0_06
- U1 pad A9: DIO0 -> GPIO_B0_07
- U1 pad B12: ENET_TX_DATA_0 -> LPSPI4_SCK
- U1 pad B13: ENET_REF_CLK -> LDO_EN
- U1 pad B14: RESET_N -> unconnected-(U1A-GPIO_B1_15-PadB14)
- U1 pad B8: LPI2C2_SDA -> GPIO_B0_05
- U1 pad B9: LPUART3_TX -> GPIO_B0_08
- U1 pad C10: unconnected-(U1A-GPIO_B0_12-PadC10) -> GPIO_B0_12
- U1 pad C12: ENET_RX_EN -> LPSPI4_SDO
- U1 pad C13: ENET_RX_ER -> PWDN
- U1 pad C14: INT_N -> EN_MAG
- U1 pad C7: ENET_MDIO -> unconnected-(U1H-GPIO_EMC_41-PadC7)
- U1 pad C8: LPI2C2_SCL -> GPIO_B0_04
- U1 pad C9: LPUART3_RX -> GPIO_B0_09
- U1 pad D11: PWM2_B_3 -> unconnected-(U1A-GPIO_B1_03-PadD11)
- U1 pad D12: ENET_RX_DATA_1 -> LPSPI4_SDI
- U1 pad D13: INH -> XRS
- U1 pad D14: WAKE -> WDT_WDI
- U1 pad D7: LPSPI4_CS -> PH2_A_3
- U1 pad D8: LPSPI4_SCK -> unconnected-(U1A-GPIO_B0_03-PadD8)
- U1 pad D9: unconnected-(U1A-GPIO_B0_10-PadD9) -> GPIO_B0_10
- U1 pad E10: unconnected-(U1A-GPIO_B0_14-PadE10) -> GPIO_B0_14
- U1 pad E11: unconnected-(U1A-GPIO_B0_15-PadE11) -> GPIO_B0_15
- U1 pad E12: ENET_RX_DATA_0 -> unconnected-(U1A-GPIO_B1_04-PadE12)
- U1 pad E14: CSI_DATA_7 -> JTAG_TMS
- U1 pad E7: LPSPI4_SDI -> PH1_B_3
- U1 pad E8: LPSPI4_SDO -> PH1_A_3
- U1 pad F12: ENET_TX_ER -> JTAG_TCK
- U1 pad F13: CSI_DATA_5 -> JTAG_MOD
- U1 pad F14: CSI_DATA_4 -> JTAG_TDI
- U1 pad G10: unconnected-(U1G-GPIO_AD_B0_11-PadG10) -> JTAG_TRSTB
- U1 pad G11: HOPERF_RST -> WDT_ENABLE
- U1 pad G12: LPSPI3_SDO -> CSI_DATA_3
- U1 pad G13: CSI_DATA_3 -> JTAG_TDO
- U1 pad G14: CSI_DATA_8 -> GPIO_AD_B0_05
- U1 pad H10: LPSPI3_CS -> LPSPI3_SDO
- U1 pad H11: ADC2_2 -> CSI_DATA_4
- U1 pad H12: ADC2_1 -> CSI_DATA_5
- U1 pad H14: CAN2_TX -> unconnected-(U1G-GPIO_AD_B0_14-PadH14)
- U1 pad J3: unconnected-(U1B-GPIO_SD_B0_01-PadJ3) -> LPI2C3_SDA
- U1 pad J4: unconnected-(U1B-GPIO_SD_B0_00-PadJ4) -> LPI2C3_SCL
- U1 pad J5: DCDC_IN -> DCDC_OUT
- U1 pad L10: CAN2_RX -> unconnected-(U1G-GPIO_AD_B0_15-PadL10)
- U1 pad L13: ADC2_15 -> CSI_DATA_7
- U1 pad L7: PMIC_STBY_REQ -> unconnected-(U1D-PMIC_STBY_REQ-PadL7)
- U1 pad M13: ADC2_14 -> CSI_DATA_8
- U1 pad M6: ONOFF -> unconnected-(U1D-ONOFF-PadM6)
- U1 pad M7: RESET -> ~{RESET}
- U5 pad 11: unconnected-(U5-DIO3-Pad11) -> GND
- U5 pad 12: DIO4 -> +1V8A
- U5 pad 13: +3.3V -> GND
- U5 pad 14: DIO0 -> Net-(U5-~{RESET})
- U5 pad 15: unconnected-(U5-DIO1-Pad15) -> GND
- U5 pad 16: unconnected-(U5-DIO2-Pad16) -> JTAG_TCK
- U5 pad 2: LPSPI3_SDO -> XCSI
- U5 pad 3: LPSPI3_SDI -> XCSO
- U5 pad 4: LPSPI3_SCK -> /USB & Debug/VPHY
- U5 pad 5: LPSPI3_CS -> GND
- U5 pad 6: HOPERF_RST -> Net-(U5-REF)
- U5 pad 7: unconnected-(U5-DIO5-Pad7) -> DM_DEBUG
- U5 pad 8: GND -> DP_DEBUG
- U5 pad 9: Net-(J8-In) -> /USB & Debug/VPLL
- U6 pad 1: CAN2_TX -> Net-(R53-Pad1)
- U6 pad 2: GND -> Net-(R51-Pad1)
- U6 pad 3: Net-(U6-VCC) -> WDT_BIAS
- U6 pad 4: CAN2_RX -> Net-(U6A--)
- U6 pad 5: SHDN -> /Watchdog/WDT-VP
- U6 pad 6: CANL -> Net-(U6B--)
- U6 pad 7: CANH -> Net-(U6B-+)
- U6 pad 8: STB -> Net-(U6C--)
Routing:
- net GND: track 81.9 -> 10.2 mm, vias 119 -> 30
- net ADC2_2: track 70.1 -> 0.00 mm, vias 1 -> 0
- net SPE_SWITCH: track 67.1 -> 0.00 mm
- net LPI2C1_SDA: track 53.5 -> 0.00 mm, vias 6 -> 1
- net LPI2C1_SCL: track 53.5 -> 0.00 mm, vias 6 -> 1
- net +3.3V: track 56.9 -> 5.96 mm, vias 74 -> 23
- net VBUS: track 47.1 -> 0.00 mm, vias 2 -> 0
- net ADC2_15: track 41.3 -> 0.00 mm, vias 1 -> 0
- net STB: track 39.6 -> 0.00 mm, vias 4 -> 0
- net ADC2_1: track 39.6 -> 0.00 mm, vias 1 -> 0
- net DIO4: track 38.6 -> 0.00 mm
- net Net-(J8-In): track 38.2 -> 0.00 mm
- net LPI2C2_SCL: track 37.9 -> 0.00 mm, vias 2 -> 0
- net CSI_DATA_8: track 37.9 -> 0.00 mm, vias 2 -> 0
- net LPI2C2_SDA: track 37.9 -> 0.00 mm, vias 2 -> 0
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- removed copper zone on In1.Cu, net (none)
- removed copper zone on F.Cu, net +3.3V
- removed copper zone on In1.Cu, net +3.3V
- removed copper zone on B.Cu, net GND
- removed copper zone on F.Cu, net GND
- removed copper zone on In2.Cu, net GND
Other:
- outline, holes or cut-outs redrawn
- board text removed: "Designed by Madhav Kapa"
- board text removed: "Project Horizon"

Commit message: finished layout of v0.2!
Parts:
- removed C53: 10uF, Capacitor_SMD:C_0402_1005Metric
- removed C54: 22uF, Capacitor_SMD:C_0603_1608Metric
- removed L4: 2.2uH, Resistor_SMD:R_0402_1005Metric
- removed R13: 100k, Resistor_SMD:R_0402_1005Metric
- removed U10: TPS62162DSG, Package_SON:WSON-8-1EP_2x2mm_P0.5mm_EP0.9x1.6mm_ThermalVias
- added C87: 10uF, Capacitor_SMD:C_0402_1005Metric, F.Cu at (81.1, 129.1)
- added C88: 22uF, Capacitor_SMD:C_0603_1608Metric, F.Cu at (80.5, 125.4)
- added H3: MountingHole, MountingHole:MountingHole_2.5mm_Pad, F.Cu at (54.1, 73.2)
- added H4: MountingHole, MountingHole:MountingHole_2.5mm_Pad, F.Cu at (104.2, 73.2)
- added H5: MountingHole, MountingHole:MountingHole_2.5mm_Pad, F.Cu at (42.5, 123.8)
- added H6: MountingHole, MountingHole:MountingHole_2.5mm_Pad, F.Cu at (42.5, 73.8)
- added H7: MountingHole, MountingHole:MountingHole_2.5mm_Pad, F.Cu at (43.4, 131.3)
- added H8: MountingHole, MountingHole:MountingHole_2.5mm_Pad, F.Cu at (98.1, 64.3)
- added H9: MountingHole, MountingHole:MountingHole_2.5mm_Pad, F.Cu at (43.1, 64.3)
- added L5: 2.2uH, Resistor_SMD:R_0402_1005Metric, F.Cu at (79.0, 126.0)
- added R66: 100k, Resistor_SMD:R_0402_1005Metric, F.Cu at (78.0, 126.0)
- added R67: 1k, Resistor_SMD:R_0402_1005Metric, B.Cu at (100.5, 79.8)
- added U11: STSPIN250, footprints:QFN50P300X300X100-17N, F.Cu at (94.8, 90.6)
- added U13: TPS62162DSG, Package_SON:WSON-8-1EP_2x2mm_P0.5mm_EP0.9x1.6mm_ThermalVias, F.Cu at (79.3, 128.5)
- added U14: PRTR5V0U2X, Package_TO_SOT_SMD:SOT-143, F.Cu at (93.0, 132.5)
- added U15: SiP32431DR3, Package_TO_SOT_SMD:SOT-363_SC-70-6, F.Cu at (99.8, 89.6)
- added U2: STSPIN250, footprints:QFN50P300X300X100-17N, F.Cu at (106.8, 91.8)
- added U8: STSPIN250, footprints:QFN50P300X300X100-17N, B.Cu at (104.4, 82.7)
- added U9: AP22652, footprints:SOT95P280X145-6N, F.Cu at (64.7, 123.4)
- C12, C16, C19, C22, C27, C28, C33, C34, C37, C38, C39, C41, C43, C47, C48, C56, C57, C58, C65, C66, C69, C70, C71, C74, C79, C83, C84, FB1, FB2, J11, L2, L3, R10, R11, R17, R20, R21, R22, R23, R24, R25, R26, R27, R28, R29, R30, R31, R32, R34, R35, R37, R38, R39, R4, R46, R48, R49, R5, R50, R52, R53, R54, R55, R56, R57, R6, R61, R9: moved to B.Cu
- C85: value 100nf -> 1uF; moved to B.Cu
- C86: value 100nf -> 0.1uF; moved to B.Cu
- J2, J4: footprint Connector_PinHeader_1.00mm:PinHeader_1x03_P1.00mm_Vertical -> Connector_PinHeader_2.54mm:PinHeader_1x03_P2.54mm_Vertical
- J6, J7: footprint Connector_PinHeader_1.00mm:PinHeader_1x02_P1.00mm_Vertical -> Connector_PinHeader_2.54mm:PinHeader_1x02_P2.54mm_Vertical
- J8: footprint Connector_PinHeader_1.00mm:PinHeader_1x04_P1.00mm_Vertical -> Connector_PinHeader_2.54mm:PinHeader_1x04_P2.54mm_Vertical
- R65: value 47k -> 10k
- moved J6 222.1 mm to (63.5, 116.1), turned to 90 degrees
- moved J8 219.3 mm to (69.6, 131.2), turned to -90 degrees
- moved J7 212.4 mm to (71.4, 90.2), turned to 90 degrees
- moved J2 207.7 mm to (83.8, 127.2), turned to 90 degrees
- moved C39 197.9 mm to (74.4, 123.2)
- moved C58 197.0 mm to (82.3, 108.2), turned to 90 degrees
- moved J4 193.6 mm to (94.8, 105.0), turned to 90 degrees
- moved C43 193.5 mm to (80.7, 112.2), turned to 90 degrees
- moved R22 193.1 mm to (89.1, 108.7), turned to 90 degrees
- moved C41 192.1 mm to (82.3, 113.0), turned to -90 degrees
- moved C37 189.7 mm to (82.0, 104.3), turned to 180 degrees
- moved C38 189.4 mm to (82.3, 106.6), turned to -90 degrees
- moved C21 186.9 mm to (83.4, 120.8)
- moved C22 186.0 mm to (83.9, 119.6), turned to -90 degrees
- moved C12 185.0 mm to (82.7, 118.0), turned to 90 degrees
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Connections:
- C13 pad 2: DCDC_IN -> +3.3V
- C14 pad 2: DCDC_IN -> +3.3V
- C16 pad 2: DCDC_IN -> +3.3V
- C17 pad 2: DCDC_IN -> +3.3V
- C18 pad 2: DCDC_IN -> +3.3V
- C86 pad 1: Net-(U24-Output) -> MAG_V
- CR2 pad 2: VBUS_FTDI -> VBUS
- J1 pad A1: Net-(J1-SHIELD) -> GND
- J1 pad A12: Net-(J1-SHIELD) -> GND
- J1 pad B1: Net-(J1-SHIELD) -> GND
- J1 pad B12: Net-(J1-SHIELD) -> GND
- J1 pad S1: Net-(J1-SHIELD) -> GND
- J3 pad 3: LPI2C3_SDA -> LPI2C4_SDA
- J3 pad 4: LPI2C3_SCL -> LPI2C4_SCL
- J6 pad 1: LPI2C4_SCL -> LPI2C3_SCL
- J6 pad 2: LPI2C4_SDA -> LPI2C3_SDA
- L3 pad 1: Net-(J1-SHIELD) -> GND
- L3 pad 2: Net-(J1-SHIELD) -> GND
- R1 pad 2: DCDC_IN -> +3.3V
- R25 pad 2: LPI2C3_SCL -> LPI2C4_SCL
- R26 pad 2: LPI2C3_SDA -> LPI2C4_SDA
- R65 pad 1: +3.3V -> REF1_A_3
- R65 pad 2: Net-(U24-ILIM) -> +3.3V
- U1 pad M9: DCDC_IN -> +3.3V
- U1 pad N14: DCDC_IN -> +3.3V
- U1 pad P12: DCDC_IN -> +3.3V
Routing:
- net GND: track 10.2 -> 185.6 mm, vias 30 -> 130
- net +3.3V: track 5.96 -> 97.5 mm, vias 23 -> 64
- net VBUS: track 0.00 -> 82.3 mm, vias 0 -> 12
- net WDT_WDI: track 0.00 -> 49.9 mm, vias 0 -> 7
- net PH1_B_3: track 0.00 -> 41.0 mm, vias 1 -> 2
- net PWM1_B_3: track 0.00 -> 39.0 mm, vias 1 -> 3
- net PH1_A_3: track 0.00 -> 37.3 mm, vias 1 -> 3
- net REF1_A_3: track 0.00 -> 36.1 mm, vias 0 -> 5
- net DP_DEBUG: track 0.00 -> 32.7 mm, vias 0 -> 2
- net DM_DEBUG: track 0.00 -> 32.7 mm, vias 0 -> 2
- net PWM1_A_3: track 0.00 -> 31.7 mm, vias 1 -> 2
- net USB_OTG1_DP: track 0.00 -> 31.2 mm
- net USB_OTG1_DN: track 0.00 -> 31.1 mm
- net GPIO_AD_B0_05: track 0.00 -> 30.6 mm, vias 0 -> 3
- net GPIO_AD_B0_04: track 0.00 -> 30.2 mm, vias 1 -> 3
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- added copper zone on In1.Cu, net +3.3V
- added copper zone on F.Cu, net DCDC_OUT
- added copper zone on In2.Cu, net GND
- added copper zone on In1.Cu, net MAG_V
- added copper zone on In1.Cu, net VBUS

Commit message: added testpoints
Parts:
- added TP10: TestPoint, TestPoint:TestPoint_Pad_D1.5mm, F.Cu at (95.6, 81.8)
- added TP4: TestPoint, TestPoint:TestPoint_Pad_D1.5mm, F.Cu at (60.0, 115.9)
- added TP5: TestPoint, TestPoint:TestPoint_Pad_D1.5mm, F.Cu at (82.5, 122.8)
- added TP6: TestPoint, TestPoint:TestPoint_Pad_D1.5mm, F.Cu at (90.3, 91.6)
- added TP7: TestPoint, TestPoint:TestPoint_Pad_D1.5mm, F.Cu at (90.3, 94.2)
- added TP8: TestPoint, TestPoint:TestPoint_Pad_D1.5mm, F.Cu at (102.5, 102.3)
- added TP9: TestPoint, TestPoint:TestPoint_Pad_D1.5mm, F.Cu at (98.7, 85.9)
Routing:
- net DCDC_OUT: track 24.5 -> 38.0 mm
- net PMIC_ON_REQ: track 0.00 -> 10.4 mm, vias 0 -> 2
- net V_POT: track 6.94 -> 15.3 mm
- net LPI2C1_SCL: track 28.6 -> 36.9 mm, vias 4 -> 5
- net REF1_A_3: track 36.1 -> 41.2 mm
- net EN_MAG: track 30.0 -> 35.1 mm
- net LPI2C1_SDA: track 26.3 -> 29.6 mm
Other:
- board text added: "DCDC_OUT (1.8V)"
- board text added: "PMIC_ON_REQ"
- board text added: "SCL"
- board text added: "SDA"
- board text added: "V_LIMIT (0.33V)"
- board text added: "V_POT"
